File: wlan.sch (KiCad schematic (older format))
At the start: 0 parts

Commit message: schematic progress
Parts:
- added C?: 22u, symbol C
- added J?: CONN-2, symbol CONN-2
- added M?: RTL8188EUS, symbol RTL8188EUS
Connections:
- new net: J?.1, M?.ANT
- new net COM: C?.2, J?.2, M?.GND
- new net PP_WLAN: C?.1, M?.3.3V
- new net USB2_DM: M?.USB_DM
- new net USB2_DP: M?.USB_DP
Changed lines of the file:
@@
 $Descr A4 11693 8268
 encoding utf-8
-Sheet 6 12
+Sheet 13 13
 Title ""
 Date ""
@@
 Comment4 ""
 $EndDescr
+Wire Wire Line
+	5300 3950 4900 3950
+Wire Wire Line
+	4900 4050 5300 4050
+Text GLabel 4900 3950 0    50   Input ~ 0
+USB2_DP
+Text GLabel 4900 4050 0    50   Input ~ 0
+USB2_DM
+$Comp
+L RTL8188EUS M?
+U 1 1 5A1FB2A9
+P 5800 3850
+F 0 "M?" H 5800 4315 50  0000 C CNN
+F 1 "RTL8188EUS" H 5800 4224 50  0000 C CNN
+F 2 "" H 5450 4250 50  0001 C CNN
+F 3 "" H 5450 4250 50  0001 C CNN
+	1    5800 3850
+	1    0    0    -1
+$EndComp
+Text GLabel 4950 3650 0    60   Input ~ 0
+PP_WLAN
+Wire Wire Line
+	4950 3650 5200 3650
+Wire Wire Line
+	5200 3650 5300 3650
+$Comp
+L C C?
+U 1 1 5A1FB3A2
+P 5200 3650
+F 0 "C?" H 5273 3596 50  0000 L CNN
+F 1 "22u" H 5273 3505 50  0000 L CNN
+F 2 "" H 5100 3800 60  0000 C CNN
+F 3 "" H 5100 3800 60  0000 C CNN
+	1    5200 3650
+	-1   0    0    -1
+$EndComp
+$Comp
+L COM #PWR?
+U 1 1 5A1FB452
+P 5200 3850
+F 0 "#PWR?" V 5475 3850 60  0001 C CNN
+F 1 "COM" H 5360 3735 30  0001 C CNN
+F 2 "" H 5355 3860 60  0000 C CNN
+F 3 "" H 5355 3860 60  0000 C CNN
+	1    5200 3850
+	1    0    0    -1
+$EndComp
+Connection ~ 5200 3650
+$Comp
+L CONN-2 J?
+U 1 1 5A1FB56A
+P 7250 3700
+F 0 "J?" H 7478 3751 50  0000 L CNN
+F 1 "CONN-2" H 7478 3660 50  0000 L CNN
+F 2 "" H 7350 3500 60  0000 C CNN
+F 3 "" H 7350 3500 60  0000 C CNN
+	1    7250 3700
+	1    0    0    -1
+$EndComp
+$Comp
+L COM #PWR?
+U 1 1 5A1FB5E6
+P 6350 4150
+F 0 "#PWR?" V 6625 4150 60  0001 C CNN
+F 1 "COM" H 6510 4035 30  0001 C CNN
+F 2 "" H 6505 4160 60  0000 C CNN
+F 3 "" H 6505 4160 60  0000 C CNN
+	1    6350 4150
+	1    0    0    -1
+$EndComp
+Wire Wire Line
+	6300 4050 6350 4050
+Wire Wire Line
+	6350 3950 6350 4050
+Wire Wire Line
+	6350 4050 6350 4150
+Wire Wire Line
+	6300 3950 6350 3950
+Connection ~ 6350 4050
+$Comp
+L COM #PWR?
+U 1 1 5A1FB67E
+P 7250 3800
+F 0 "#PWR?" V 7525 3800 60  0001 C CNN
+F 1 "COM" H 7410 3685 30  0001 C CNN
+F 2 "" H 7405 3810 60  0000 C CNN
+F 3 "" H 7405 3810 60  0000 C CNN
+	1    7250 3800
+	1    0    0    -1
+$EndComp
+Wire Wire Line
+	7250 3750 7250 3800
+Wire Wire Line
+	7250 3650 6300 3650
 $EndSCHEMATC
