File: almond.sch (KiCad schematic (older format))
At the start: 0 parts

Commit message: ddr, emmc, sd
Other:
- note added: "eMMC\nSD"
Changed lines of the file:
@@
 EESchema Schematic File Version 3
+LIBS:ap24x1-u-dfn3030
+LIBS:fpf1321
+LIBS:emmc-100fbga
 LIBS:ddr3-96fbga
 LIBS:mcimx6y2dvm
@@
 Text Notes 4250 3450 0    200  ~ 40
 DDR3
+Text Notes 6250 3750 0    200  ~ 40
+eMMC\nSD
 $EndSCHEMATC

Commit message: add control
Other:
- note added: "i.MX6\nControl"
Changed lines of the file:
@@
 $Descr A4 11693 8268
 encoding utf-8
-Sheet 1 10
+Sheet 1 11
 Title "Almond"
 Date "2017-11-02"
@@
 Text Notes 6250 3750 0    200  ~ 40
 eMMC\nSD
+$Sheet
+S 4000 950  1450 1350
+U 5A0FEE94
+F0 "imx6control" 50
+F1 "imx6control.sch" 50
+$EndSheet
+Text Notes 4150 1900 0    200  ~ 40
+i.MX6\nControl
 $EndSCHEMATC

Commit message: start some usb
Other:
- note added: "USB"
Changed lines of the file:
@@
 Text Notes 4150 1900 0    200  ~ 40
 i.MX6\nControl
+Text Notes 4250 5300 0    200  ~ 40
+USB
 $EndSCHEMATC

Commit message: schematic progress
Other:
- note added: "SD"
- note added: "USB\nWLAN"
- note added: "eMMC"
- note removed: "USB"
- note removed: "eMMC\nSD"
Changed lines of the file:
@@
 EESchema Schematic File Version 3
+LIBS:tpd3s014
+LIBS:rtl8188eus
 LIBS:ap24x1-u-dfn3030
 LIBS:fpf1321
@@
 $Descr A4 11693 8268
 encoding utf-8
-Sheet 1 11
+Sheet 1 12
 Title "Almond"
 Date "2017-11-02"
@@
 $EndSheet
 $Sheet
-S 8000 2800 1450 1350
+S 2000 6500 1450 1350
 U 59FBAC53
 F0 "periph" 60
@@
 Text Notes 4250 3450 0    200  ~ 40
 DDR3
-Text Notes 6250 3750 0    200  ~ 40
-eMMC\nSD
+Text Notes 6250 3450 0    200  ~ 40
+eMMC
 $Sheet
 S 4000 950  1450 1350
@@
 Text Notes 4150 1900 0    200  ~ 40
 i.MX6\nControl
-Text Notes 4250 5300 0    200  ~ 40
-USB
+Text Notes 4250 5600 0    200  ~ 40
+USB\nWLAN
+$Sheet
+S 8000 2800 1450 1350
+U 5A1F2DC0
+F0 "sd" 60
+F1 "sd.sch" 60
+$EndSheet
+Text Notes 8250 3450 0    200  ~ 40
+SD
 $EndSCHEMATC

Commit message: power design
Other:
- note added: "Power"
- note added: "XXX replace NUP4114 with D1213A-04S"
Changed lines of the file:
@@
-EESchema Schematic File Version 3
-LIBS:tpd3s014
-LIBS:rtl8188eus
-LIBS:ap24x1-u-dfn3030
-LIBS:fpf1321
-LIBS:emmc-100fbga
-LIBS:ddr3-96fbga
-LIBS:mcimx6y2dvm
-LIBS:zener
-LIBS:xtal
-LIBS:vutmi
-LIBS:vusb
-LIBS:vtarget
-LIBS:vpll
-LIBS:vout
-LIBS:vio
-LIBS:vin
-LIBS:vcore
-LIBS:vbu
-LIBS:varef
-LIBS:vana
-LIBS:usb334x
-LIBS:usb
-LIBS:usb-c
-LIBS:ts3usb31
-LIBS:tps6040x
-LIBS:tps27081a
-LIBS:tpd4s012
-LIBS:tp4056
-LIBS:tp4055
-LIBS:tlv713
-LIBS:thermistor
-LIBS:testpoint
-LIBS:test
-LIBS:tactile-4
-LIBS:spiflash
-LIBS:solder-jumper-nc
-LIBS:slide-spdt
-LIBS:sit1602
-LIBS:sip32401a
-LIBS:si8410
-LIBS:schottky
-LIBS:rs485trx-fullduplex
-LIBS:relay
-LIBS:r4
-LIBS:r
-LIBS:pwr
-LIBS:powersyms
-LIBS:power_flag
-LIBS:pot
-LIBS:pnp
-LIBS:pmos
-LIBS:phone-3
-LIBS:op-amp
-LIBS:nup4114
-LIBS:npn
-LIBS:nmos
-LIBS:nmos-pmos-sot23-6
-LIBS:nmos-pmos-sot-666
-LIBS:mun53
-LIBS:mpu6050
-LIBS:mpu-6050
-LIBS:mpl3115a2
-LIBS:mounting-hole
-LIBS:mounthole
-LIBS:mkl27zxxvfm4
-LIBS:mkl03zxxvfk4
-LIBS:mkl03zxxvfg4
-LIBS:microsd
-LIBS:mic9409x
-LIBS:mic5365
-LIBS:mic5205
-LIBS:mic23031
-LIBS:mcp47x6-sot-23-6
-LIBS:mcp3221
-LIBS:mchck
-LIBS:max9938
-LIBS:max6070
-LIBS:max4737eud
-LIBS:mag3110
-LIBS:ltc3260
-LIBS:ltc3251
-LIBS:lt6106
-LIBS:lt6102
-LIBS:lpddrx16
-LIBS:lpc824
-LIBS:lpc812
-LIBS:ln1410
-LIBS:lm78xx-so8
-LIBS:lm3671
-LIBS:lm27313
-LIBS:lis2-lga12
-LIBS:led
-LIBS:ldo-sot-23-5
-LIBS:lcd5110
-LIBS:l
-LIBS:k22f-64lqfp
-LIBS:jumper
-LIBS:jtag
-LIBS:isp130301
-LIBS:ip425xcz12
-LIBS:ina199
-LIBS:in-amp
-LIBS:gnd
-LIBS:fuse
-LIBS:ferrite
-LIBS:esp-12
-LIBS:erc12864-1
-LIBS:dtc-npn
-LIBS:drv883x
-LIBS:drv8839
-LIBS:drv8838
-LIBS:drdc3105
-LIBS:debugheader
-LIBS:de-9
-LIBS:d
-LIBS:cp
-LIBS:conn-8
-LIBS:conn-7
-LIBS:conn-6
-LIBS:conn-5
-LIBS:conn-4
-LIBS:conn-3
-LIBS:conn-2x5
-LIBS:conn-2x4
-LIBS:conn-2
-LIBS:conn-1
-LIBS:com
-LIBS:cm1624
-LIBS:c
-LIBS:button-dpdt
-LIBS:buck-sot23-6
-LIBS:buck-sot23-5
-LIBS:bat
-LIBS:ant
-LIBS:ad8429
-LIBS:acs711ex
-LIBS:aat3681a
-LIBS:aat1217
-LIBS:USB3300
-LIBS:SAM3U-144
-LIBS:MKL26ZxxVFM4
-LIBS:ICE40HX4K-144
-LIBS:74vc2t45
-LIBS:74vc1t45
-LIBS:74avc4t245
-LIBS:2-spst
-LIBS:-vs
-LIBS:-15v
-LIBS:+vs
-LIBS:+5v
-LIBS:+3v3
-LIBS:+3v
-LIBS:+1v8
-LIBS:+1v2
-LIBS:+15v
-LIBS:+12v
+EESchema Schematic File Version 4
 LIBS:almond-cache
 EELAYER 26 0
@@
 Text Notes 8250 3450 0    200  ~ 40
 SD
+Text Notes 8250 5250 0    200  ~ 40
+Power
+Text Notes 7950 1100 0    50   ~ 0
+XXX replace NUP4114 with D1213A-04S
 $EndSCHEMATC
