File: ddr3.sch (KiCad schematic (older format))
At the start: 17 parts

Commit message: add ddr3
Parts:
- added C? (x7): 0.22u, symbol C
- added C?: 22u, symbol C
- added C? (x4): 2.2p, symbol C
- added R?: 240, symbol R
- added R?: 470, symbol R
- added TP? (x2): A0, symbol TESTPOINT
- added TP? (x2): DQ0, symbol TESTPOINT
- added TP? (x2): CK, symbol TESTPOINT
- added TP? (x2): ~CK, symbol TESTPOINT
- added TP? (x4): GND, symbol TESTPOINT
- added U?: MT41K256M16-107, symbol DDR3-96FBGA
- R?: value Rs -> 10k; symbol Rs -> R
Connections:
- net labels added: DRAM_A0, DRAM_A1, DRAM_A10, DRAM_A11, DRAM_A12, DRAM_A13, DRAM_A14, DRAM_A2, DRAM_A3, DRAM_A4, DRAM_A5, DRAM_A6, DRAM_A7, DRAM_A8, DRAM_A9, DRAM_A[14:0],DRAM_BA[2:0],DRAM_CONTROL, DRAM_BA0, DRAM_BA1, DRAM_BA2, DRAM_CK, DRAM_CKE, DRAM_DATA[15:0],DRAM_DQ,DRAM_DM, DRAM_DQ0, DRAM_DQ1, DRAM_DQ10, DRAM_DQ11, DRAM_DQ12, DRAM_DQ13, DRAM_DQ14, DRAM_DQ15, DRAM_DQ2, DRAM_DQ3, DRAM_DQ4, DRAM_DQ5, DRAM_DQ6, DRAM_DQ7, DRAM_DQ8, DRAM_DQ9, DRAM_LDM, DRAM_LDQS, DRAM_ODT, DRAM_UDM, DRAM_UDQS, ~DRAM_CAS, ~DRAM_CK, ~DRAM_CS, ~DRAM_LDQS, ~DRAM_RAS, ~DRAM_RESET, ~DRAM_UDQS, ~DRAM_WE
- wire segments 38 -> 209
- no-connect marks 0 -> 4
Other:
- note added: "DRAM Termination"
- note added: "DRAM VREF"
- note added: "Signal Integrity"
- note added: "place close to DRAM IC"
- note added: "place close to SoC"
- moved on the sheet: C?, R?, U?B

Commit message: ddr, emmc, sd
Parts:
- added C? (x6): 0.22u, symbol C
Connections:
- net COM: now also C?.2, C?.2, C?.2, C?.2, C?.2, C?.2
- net PP_DRAM: now also C?.1, C?.1, C?.1, C?.1, C?.1, C?.1
Other:
- moved on the sheet: C?, R?, TP?, U?

Commit message: power design
Parts:
- C301, C302, C303, C304, C306, C307, C308, C309, C310, C311, C312, C313, C314, C315, C316, C317, C318, C319, C320, C321, C322, C324, C330: renamed from C?; footprint (none) -> kicad-libs:SMD-1005; symbol C -> c:C; Manufacturer (none) -> Samsung; Part Number (none) -> CL05B224KQ5NNWC
- C305: renamed from C?; footprint (none) -> kicad-libs:SMD-1608; symbol C -> c:C; Manufacturer (none) -> Samsung; Part Number (none) -> CL10A226MQ8NRNC
- C323: renamed from C?; footprint (none) -> kicad-libs:SMD-1608; symbol C -> c:C; Manufacturer (none) -> Samsung; Part Number (none) -> CL10A106MQ8NNNC
- C325: renamed from C?; value 4.7u -> 10u; footprint (none) -> kicad-libs:SMD-1005; symbol C -> c:C; Manufacturer (none) -> Murata; Part Number (none) -> GRM155R60G106ME44D
- C326, C327, C328, C329: renamed from C?; symbol C -> c:C
- R301, R302, R303, R304, R305, R306: renamed from R?; symbol R -> r:R
- TP301, TP302, TP303, TP304, TP305, TP306, TP307, TP308, TP309, TP310, TP311, TP312: renamed from TP?; symbol TESTPOINT -> testpoint:TESTPOINT
- U201: renamed from U?; symbol MCIMX6Y2DVM -> mcimx6y2dvm:MCIMX6Y2DVM
- U301: renamed from U?; symbol DDR3-96FBGA -> ddr3-96fbga:DDR3-96FBGA
