File: fpga.sch (KiCad schematic (older format))
At the start: 0 parts

Commit message: add control
Parts:
- added U? (x2): MCIMX6Y2DVM, symbol MCIMX6Y2DVM
Changed lines of the file:
@@
 $Descr A4 11693 8268
 encoding utf-8
-Sheet 1 10
+Sheet 8 11
 Title ""
 Date ""
@@
 Comment4 ""
 $EndDescr
+$Comp
+L MCIMX6Y2DVM U?
+U 9 1 5A0FEC80
+P 3900 1700
+F 0 "U?" H 3900 1987 60  0000 C CNN
+F 1 "MCIMX6Y2DVM" H 3900 1881 60  0000 C CNN
+F 2 "" H 1750 700 60  0001 C CNN
+F 3 "" H 1750 700 60  0001 C CNN
+	9    3900 1700
+	1    0    0    -1
+$EndComp
+$Comp
+L MCIMX6Y2DVM U?
+U 10 1 5A0FEE00
+P 3900 4200
+F 0 "U?" H 3900 4487 60  0000 C CNN
+F 1 "MCIMX6Y2DVM" H 3900 4381 60  0000 C CNN
+F 2 "" H 1750 3200 60  0001 C CNN
+F 3 "" H 1750 3200 60  0001 C CNN
+	10   3900 4200
+	1    0    0    -1
+$EndComp
 $EndSCHEMATC

Commit message: power design
Parts:
- U201: renamed from U?; symbol MCIMX6Y2DVM -> mcimx6y2dvm:MCIMX6Y2DVM
Other:
- note added: "ICE40 HX 132 csBGA"
Changed lines of the file:
@@
-EESchema Schematic File Version 3
-LIBS:tpd3s014
-LIBS:rtl8188eus
-LIBS:ap24x1-u-dfn3030
-LIBS:fpf1321
-LIBS:emmc-100fbga
-LIBS:ddr3-96fbga
-LIBS:mcimx6y2dvm
-LIBS:zener
-LIBS:xtal
-LIBS:vutmi
-LIBS:vusb
-LIBS:vtarget
-LIBS:vpll
-LIBS:vout
-LIBS:vio
-LIBS:vin
-LIBS:vcore
-LIBS:vbu
-LIBS:varef
-LIBS:vana
-LIBS:usb334x
-LIBS:usb
-LIBS:usb-c
-LIBS:ts3usb31
-LIBS:tps6040x
-LIBS:tps27081a
-LIBS:tpd4s012
-LIBS:tp4056
-LIBS:tp4055
-LIBS:tlv713
-LIBS:thermistor
-LIBS:testpoint
-LIBS:test
-LIBS:tactile-4
-LIBS:spiflash
-LIBS:solder-jumper-nc
-LIBS:slide-spdt
-LIBS:sit1602
-LIBS:sip32401a
-LIBS:si8410
-LIBS:schottky
-LIBS:rs485trx-fullduplex
-LIBS:relay
-LIBS:r4
-LIBS:r
-LIBS:pwr
-LIBS:powersyms
-LIBS:power_flag
-LIBS:pot
-LIBS:pnp
-LIBS:pmos
-LIBS:phone-3
-LIBS:op-amp
-LIBS:nup4114
-LIBS:npn
-LIBS:nmos
-LIBS:nmos-pmos-sot23-6
-LIBS:nmos-pmos-sot-666
-LIBS:mun53
-LIBS:mpu6050
-LIBS:mpu-6050
-LIBS:mpl3115a2
-LIBS:mounting-hole
-LIBS:mounthole
-LIBS:mkl27zxxvfm4
-LIBS:mkl03zxxvfk4
-LIBS:mkl03zxxvfg4
-LIBS:microsd
-LIBS:mic9409x
-LIBS:mic5365
-LIBS:mic5205
-LIBS:mic23031
-LIBS:mcp47x6-sot-23-6
-LIBS:mcp3221
-LIBS:mchck
-LIBS:max9938
-LIBS:max6070
-LIBS:max4737eud
-LIBS:mag3110
-LIBS:ltc3260
-LIBS:ltc3251
-LIBS:lt6106
-LIBS:lt6102
-LIBS:lpddrx16
-LIBS:lpc824
-LIBS:lpc812
-LIBS:ln1410
-LIBS:lm78xx-so8
-LIBS:lm3671
-LIBS:lm27313
-LIBS:lis2-lga12
-LIBS:led
-LIBS:ldo-sot-23-5
-LIBS:lcd5110
-LIBS:l
-LIBS:k22f-64lqfp
-LIBS:jumper
-LIBS:jtag
-LIBS:isp130301
-LIBS:ip425xcz12
-LIBS:ina199
-LIBS:in-amp
-LIBS:gnd
-LIBS:fuse
-LIBS:ferrite
-LIBS:esp-12
-LIBS:erc12864-1
-LIBS:dtc-npn
-LIBS:drv883x
-LIBS:drv8839
-LIBS:drv8838
-LIBS:drdc3105
-LIBS:debugheader
-LIBS:de-9
-LIBS:d
-LIBS:cp
-LIBS:conn-8
-LIBS:conn-7
-LIBS:conn-6
-LIBS:conn-5
-LIBS:conn-4
-LIBS:conn-3
-LIBS:conn-2x5
-LIBS:conn-2x4
-LIBS:conn-2
-LIBS:conn-1
-LIBS:com
-LIBS:cm1624
-LIBS:c
-LIBS:button-dpdt
-LIBS:buck-sot23-6
-LIBS:buck-sot23-5
-LIBS:bat
-LIBS:ant
-LIBS:ad8429
-LIBS:acs711ex
-LIBS:aat3681a
-LIBS:aat1217
-LIBS:USB3300
-LIBS:SAM3U-144
-LIBS:MKL26ZxxVFM4
-LIBS:ICE40HX4K-144
-LIBS:74vc2t45
-LIBS:74vc1t45
-LIBS:74avc4t245
-LIBS:2-spst
-LIBS:-vs
-LIBS:-15v
-LIBS:+vs
-LIBS:+5v
-LIBS:+3v3
-LIBS:+3v
-LIBS:+1v8
-LIBS:+1v2
-LIBS:+15v
-LIBS:+12v
+EESchema Schematic File Version 4
 LIBS:almond-cache
 EELAYER 26 0
@@
 $EndDescr
 $Comp
-L MCIMX6Y2DVM U?
+L mcimx6y2dvm:MCIMX6Y2DVM U201
 U 9 1 5A0FEC80
 P 3900 1700
-F 0 "U?" H 3900 1987 60  0000 C CNN
+F 0 "U201" H 3900 1987 60  0000 C CNN
 F 1 "MCIMX6Y2DVM" H 3900 1881 60  0000 C CNN
 F 2 "" H 1750 700 60  0001 C CNN
@@
 $EndComp
 $Comp
-L MCIMX6Y2DVM U?
+L mcimx6y2dvm:MCIMX6Y2DVM U201
 U 10 1 5A0FEE00
 P 3900 4200
-F 0 "U?" H 3900 4487 60  0000 C CNN
+F 0 "U201" H 3900 4487 60  0000 C CNN
 F 1 "MCIMX6Y2DVM" H 3900 4381 60  0000 C CNN
 F 2 "" H 1750 3200 60  0001 C CNN
@@
 	1    0    0    -1
 $EndComp
+Text Notes 7800 2600 0    50   ~ 0
+ICE40 HX 132 csBGA
 $EndSCHEMATC
