File: power.sch (KiCad schematic (older format))
At the start: 0 parts

Commit message: add schematic sheets, fix pins
Other:
- note removed: "DDR3"
- note removed: "i.MX6\nPower"
Changed lines of the file:
@@
 $Descr A4 11693 8268
 encoding utf-8
-Sheet 1 10
-Title "Almond"
-Date "2017-11-02"
-Rev "0"
-Comp "Sternlabs"
+Sheet 3 10
+Title ""
+Date ""
+Rev ""
+Comp ""
 Comment1 ""
 Comment2 ""
@@
 Comment4 ""
 $EndDescr
-$Sheet
-S 2000 2800 1450 1350
-U 59FBAA99
-F0 "imx6power" 60
-F1 "imx6power.sch" 60
-$EndSheet
-$Sheet
-S 4000 2800 1450 1350
-U 59FBAAE5
-F0 "ddr3" 60
-F1 "ddr3.sch" 60
-$EndSheet
-$Sheet
-S 6000 2800 1450 1350
-U 59FBAAF4
-F0 "emmc" 60
-F1 "emmc.sch" 60
-$EndSheet
-$Sheet
-S 4000 4650 1450 1350
-U 59FBAC0A
-F0 "usb" 60
-F1 "usb.sch" 60
-$EndSheet
-$Sheet
-S 8000 2800 1450 1350
-U 59FBAC53
-F0 "periph" 60
-F1 "periph.sch" 60
-$EndSheet
-$Sheet
-S 2000 4650 1450 1350
-U 59FBACC1
-F0 "rampscontrol" 60
-F1 "rampscontrol.sch" 60
-$EndSheet
-$Sheet
-S 6000 4650 1450 1350
-U 59FBABF8
-F0 "fpga" 60
-F1 "fpga.sch" 60
-$EndSheet
-$Sheet
-S 8000 4650 1450 1350
-U 59FBAAD3
-F0 "power" 60
-F1 "power.sch" 60
-$EndSheet
-Text Notes 2250 3650 0    200  ~ 40
-i.MX6\nPower
-$Sheet
-S 2000 950  1450 1350
-U 5A04ED2D
-F0 "powernets" 60
-F1 "powernets.sch" 60
-$EndSheet
-Text Notes 4250 3450 0    200  ~ 40
-DDR3
 $EndSCHEMATC

Commit message: power design
Parts:
- added C901, C908: 47u, symbol cp:CP
- added C902, C903, C906, C907: 10u, kicad-libs:SMD-3216, symbol c:C
- added C904, C905: 0.22u, kicad-libs:SMD-1005, symbol c:C
- added C909: 18p, symbol c:C
- added C910: 6.8n, symbol c:C
- added C911, C912, C914, C915, C917, C918: 10u, kicad-libs:SMD-2012, symbol c:C
- added C913, C916, C919: 22p, symbol c:C
- added C920, C921, C922, C923: 10u, kicad-libs:SMD-1608, symbol c:C
- added L901: 6.8u, kicad-libs:SMD-L-6060, symbol l:L
- added L902, L903, L904: 2.2u, kicad-libs:SMD-2520, symbol l:L
- added R901: 430k, symbol r:Rs
- added R902: 82k, symbol r:Rs
- added R903: 15k, symbol r:Rs
- added R904, R907, R909: 300k, symbol r:Rs
- added R905: 66.5k, symbol r:Rs
- added R906: 100k, symbol r:R
- added R908: 226k, symbol r:Rs
- added R910: 240k, symbol r:Rs
- added U901: BD9E302EFJ, kicad-libs:SOIC-8-N-EP, symbol bd9e302efj:BD9E302EFJ
- added U902, U903, U904: AP3402, kicad-libs:SOT-23-6, symbol AP3402:AP3402
- added U905: MIC5365-1.8, kicad-libs:SC-70-5, symbol mic5365:MIC5365
- added U906: MIC5365-1.2, kicad-libs:SC-70-5, symbol mic5365:MIC5365
Connections:
- net labels added: COM, PGOOD_3V3, PP_1V2, PP_1V35, PP_1V4, PP_1V8, PP_24V, PP_3V3, PP_5V
- wire segments 0 -> 73
- no-connect marks 0 -> 4
Other:
- note added: "1.4A"
- note added: "2.7A"
- note added: "31m"
- note added: "325mA"
- note added: "400m"
- note added: "75mA"
- note added: "reduce comp R to improve stability"
