File: powernets.sch (KiCad schematic (older format))
At the start: 0 parts

Commit message: add schematic sheets, fix pins
Other:
- note removed: "DDR3"
- note removed: "i.MX6\nPower"
Changed lines of the file:
@@
 $Descr A4 11693 8268
 encoding utf-8
-Sheet 1 10
-Title "Almond"
-Date "2017-11-02"
-Rev "0"
-Comp "Sternlabs"
+Sheet 10 10
+Title ""
+Date ""
+Rev ""
+Comp ""
 Comment1 ""
 Comment2 ""
@@
 Comment4 ""
 $EndDescr
-$Sheet
-S 2000 2800 1450 1350
-U 59FBAA99
-F0 "imx6power" 60
-F1 "imx6power.sch" 60
-$EndSheet
-$Sheet
-S 4000 2800 1450 1350
-U 59FBAAE5
-F0 "ddr3" 60
-F1 "ddr3.sch" 60
-$EndSheet
-$Sheet
-S 6000 2800 1450 1350
-U 59FBAAF4
-F0 "emmc" 60
-F1 "emmc.sch" 60
-$EndSheet
-$Sheet
-S 4000 4650 1450 1350
-U 59FBAC0A
-F0 "usb" 60
-F1 "usb.sch" 60
-$EndSheet
-$Sheet
-S 8000 2800 1450 1350
-U 59FBAC53
-F0 "periph" 60
-F1 "periph.sch" 60
-$EndSheet
-$Sheet
-S 2000 4650 1450 1350
-U 59FBACC1
-F0 "rampscontrol" 60
-F1 "rampscontrol.sch" 60
-$EndSheet
-$Sheet
-S 6000 4650 1450 1350
-U 59FBABF8
-F0 "fpga" 60
-F1 "fpga.sch" 60
-$EndSheet
-$Sheet
-S 8000 4650 1450 1350
-U 59FBAAD3
-F0 "power" 60
-F1 "power.sch" 60
-$EndSheet
-Text Notes 2250 3650 0    200  ~ 40
-i.MX6\nPower
-$Sheet
-S 2000 950  1450 1350
-U 5A04ED2D
-F0 "powernets" 60
-F1 "powernets.sch" 60
-$EndSheet
-Text Notes 4250 3450 0    200  ~ 40
-DDR3
 $EndSCHEMATC
