File: sd.sch (KiCad schematic (older format))
At the start: 20 parts

Commit message: power design
Parts:
- C1201: renamed from C?; footprint (none) -> kicad-libs:SMD-1608; symbol C -> c:C; Manufacturer (none) -> Samsung; Part Number (none) -> CL10A226MQ8NRNC
- C1202, C1204: renamed from C?; footprint (none) -> kicad-libs:SMD-1005; symbol C -> c:C; Manufacturer (none) -> Samsung; Part Number (none) -> CL05B224KQ5NNWC
- C1203: renamed from C?; value 2.2u -> 10u; footprint (none) -> kicad-libs:SMD-1005; symbol C -> c:C; Manufacturer (none) -> Murata; Part Number (none) -> GRM155R60G106ME44D
- J1201: renamed from J?; symbol MICROSD-DET -> microsd:MICROSD-DET
- R1201, R1202, R1203, R1204, R1205, R1206, R1207, R1208, R1209, R1210: renamed from R?; symbol R -> r:R
- U1201: renamed from U?; symbol FPF1321 -> fpf1321:FPF1321
- U1202: renamed from U?; symbol AP24x1-U-DFN3030 -> ap24x1-u-dfn3030:AP24x1-U-DFN3030
- U1203, U1204: renamed from U?; symbol NUP4114 -> nup4114:NUP4114
- U201: renamed from U?; symbol MCIMX6Y2DVM -> mcimx6y2dvm:MCIMX6Y2DVM
Connections:
- net PP_GPIO renamed PP_UART
Other:
- note added: "XXX add SD header"
- moved on the sheet: C1203
